Commit message: raising the robot's base link to avoid collisions with the ground

File: src/universal_robot/ur_description/urdf/ur5_joint_limited_robot.urdf.xacro (robot description, xacro)
@@ -21,5 +21,5 @@
     <parent link="world" />
     <child link = "base_link" />
-    <origin xyz="0.0 0.0 0.0" rpy="0.0 0.0 0.0" />
+    <origin xyz="0.0 0.0 2.0" rpy="0.0 0.0 0.0" />
   </joint>
 </robot>
